Commit message: UR-SIM

File: src/universal_robot/ur_e_description/urdf/common.gazebo.xacro (robot description, xacro)
@@ -3,6 +3,7 @@
   <gazebo>
     <plugin name="ros_control" filename="libgazebo_ros_control.so">
-      <!--robotNamespace>/</robotNamespace-->
-      <!--robotSimType>gazebo_ros_control/DefaultRobotHWSim</robotSimType-->
+      <robotNamespace>/</robotNamespace>
+      <robotSimType>gazebo_ros_control/DefaultRobotHWSim</robotSimType>
+      <legacyModeNS>true</legacyModeNS>
     </plugin>
 <!--

File: src/universal_robot/ur_e_description/urdf/ur5e.urdf.xacro (robot description, xacro)
@@ -1,5 +1,5 @@
 <?xml version="1.0"?>
 <robot xmlns:xacro="http://ros.org/wiki/xacro">
-  <xacro:include filename="$(find ur_e_description)/urdf/ur.transmission.xacro" />
+  <xacro:include filename="$(find ur_e_description)/urdf/ur.transmission.velocity.xacro" />
   <xacro:include filename="$(find ur_e_description)/urdf/ur.gazebo.xacro" />
   <xacro:macro name="cylinder_inertial" params="radius length mass *origin">

File: src/universal_robot/ur_e_description/urdf/ur5e_robot.urdf.xacro (robot description, xacro)
@@ -17,5 +17,4 @@
   <xacro:include filename="$(find robotiq_3f_gripper_visualization)/cfg/robotiq-3f-gripper_articulated_macro.xacro" />
   <xacro:robotiq-3f-gripper_articulated prefix="3f_gripper_"/>
-  <!-- </xacro:macro> -->
   <joint name="gripper_palm_joint" type="fixed">
     <parent link="ee_link" />
@@ -23,3 +22,4 @@
     <origin xyz="0.050 0.0 0.0" rpy="0.0 0.0 -1.57079632679" />
   </joint>
+  <!-- </xacro:macro> -->
 </robot>
