Commit message: velocity control

File: src/universal_robot/ur_e_description/urdf/ur5e_robot.urdf.xacro (robot description, xacro)
@@ -9,7 +9,13 @@
   <!-- arm -->
   <xacro:ur5e_robot prefix="" joint_limited="false"/>
-  <link name="world" />
+  <!-- <link name="world" />
   <joint name="world_joint" type="fixed">
     <parent link="world" />
+    <child link = "base_link" />
+    <origin xyz="0.0 0.0 0.0" rpy="0.0 0.0 0.0" />
+  </joint> -->
+  <link name="robot_base" />
+  <joint name="world_joint" type="fixed">
+    <parent link="robot_base" />
     <child link = "base_link" />
     <origin xyz="0.0 0.0 0.0" rpy="0.0 0.0 0.0" />
